Commit message: modify

File: piper_study_description/urdf/piper_description.xacro (robot description, xacro)
@@ -429,13 +429,18 @@
     </visual>
     <collision>
-      <origin
-        xyz="0 0 0"
-        rpy="0 0 0" />
-      <geometry>
-        <mesh
-          filename="package://piper_description/meshes/link7.STL" />
-      </geometry>
-    </collision>
-  </link>
+      <max_contacts>30</max_contacts>
+      <origin xyz="0 -0.03 -0.005" rpy="0 0 0" />
+      <geometry>
+        <box size="0.10 0.07 0.01" />
+      </geometry>
+    </collision>
+  </link>
+  <gazebo reference="link7">
+    <implicitSpringDamper>1</implicitSpringDamper>
+    <mu1>100000</mu1>
+    <mu2>100000</mu2>
+    <kp>100000000.0</kp>
+    <kd>1.0</kd>
+  </gazebo>
   <joint
     name="joint7"
@@ -453,5 +458,5 @@
       lower="0"
       upper="0.04"
-      effort="10"
+      effort="100"
       velocity="1" />
   </joint>
@@ -487,13 +492,18 @@
     </visual>
     <collision>
-      <origin
-        xyz="0 0 0"
-        rpy="0 0 0" />
-      <geometry>
-        <mesh
-          filename="package://piper_description/meshes/link8.STL" />
-      </geometry>
-    </collision>
-  </link>
+      <max_contacts>30</max_contacts>
+      <origin xyz="0 0.03 -0.005" rpy="0 0 0" />
+      <geometry>
+        <box size="0.10 0.07 0.01" />
+      </geometry>
+    </collision>
+  </link>
+  <gazebo reference="link8">
+    <implicitSpringDamper>1</implicitSpringDamper>
+    <mu1>100000</mu1>
+    <mu2>100000</mu2>
+    <kp>100000000.0</kp>
+    <kd>1.0</kd>
+  </gazebo>
   <joint
     name="joint8"
@@ -511,7 +521,14 @@
       lower="-0.04"
       upper="0"
-      effort="10"
+      effort="100"
       velocity="1" />
   </joint>
+  <gazebo>
+    <plugin filename="libgazebo_mimic_joint_plugin.so" name="mimic_joint7_to_joint8">
+      <joint>joint7</joint>
+      <mimicJoint>joint8</mimicJoint>
+      <multiplier>-1.0</multiplier>
+    </plugin>
+  </gazebo>
 <!-- controller -->
   <xacro:macro name="transmission_block" params="tran_name joint_name motor_name">

Commit message: pick and place

File: piper_study_description/urdf/piper_description.xacro (robot description, xacro)
@@ -107,4 +107,5 @@
       effort="100"
       velocity="3" />
+    <dynamics damping="0.0" friction="0.0" />
   </joint>
   <link
@@ -165,4 +166,5 @@
       effort="100"
       velocity="3" />
+    <dynamics damping="0.0" friction="0.0" />
   </joint>
   <link
@@ -223,4 +225,5 @@
       effort="100"
       velocity="3" />
+    <dynamics damping="0.0" friction="0.0" />
   </joint>
   <link
@@ -281,4 +284,5 @@
       effort="100"
       velocity="3" />
+    <dynamics damping="0.0" friction="0.0" />
   </joint>
   <link
@@ -339,4 +343,5 @@
       effort="100"
       velocity="3" />
+    <dynamics damping="0.0" friction="0.0" />
   </joint>
   <link
@@ -397,4 +402,5 @@
       effort="100"
       velocity="3" />
+    <dynamics damping="0.0" friction="0.0" />
   </joint>
   <link
@@ -437,9 +443,9 @@
   </link>
   <gazebo reference="link7">
-    <implicitSpringDamper>1</implicitSpringDamper>
-    <mu1>100000</mu1>
-    <mu2>100000</mu2>
-    <kp>100000000.0</kp>
+    <kp>1000000.0</kp>
     <kd>1.0</kd>
+    <mu1>1.0</mu1>
+    <mu2>1.0</mu2>
+    <minDepth>0.001</minDepth>
   </gazebo>
   <joint
@@ -460,4 +466,5 @@
       effort="100"
       velocity="1" />
+    <dynamics damping="0.0" friction="0.0" />
   </joint>
   <link
@@ -500,9 +507,9 @@
   </link>
   <gazebo reference="link8">
-    <implicitSpringDamper>1</implicitSpringDamper>
-    <mu1>100000</mu1>
-    <mu2>100000</mu2>
-    <kp>100000000.0</kp>
+    <kp>1000000.0</kp>
     <kd>1.0</kd>
+    <mu1>1.0</mu1>
+    <mu2>1.0</mu2>
+    <minDepth>0.001</minDepth>
   </gazebo>
   <joint
@@ -523,4 +530,5 @@
       effort="100"
       velocity="1" />
+    <dynamics damping="0.0" friction="0.0" />
   </joint>
   <gazebo>
@@ -536,8 +544,8 @@
         <type>transmission_interface/SimpleTransmission</type>
         <joint name="${joint_name}">
-            <hardwareInterface>hardware_interface/PositionJointInterface</hardwareInterface>
+            <hardwareInterface>hardware_interface/EffortJointInterface</hardwareInterface>
         </joint>
         <actuator name="$motor_name">
-            <hardwareInterface>hardware_interface/PositionJointInterface</hardwareInterface>
+            <hardwareInterface>hardware_interface/EffortJointInterface</hardwareInterface>
             <mechanicalReduction>1</mechanicalReduction>
         </actuator>
